Commit message: fixed performance issues

File: urdf/hexpet.xacro (robot description, xacro)
@@ -17,5 +17,5 @@
             <origin xyz="0.0 0.0 0.0" rpy="0.0 0.0 0.0"/>
             <geometry>
-                <box size="${body_length_x} ${body_length_y} 0.1"/>
+                <mesh filename="package://hexpet/meshes/phantomX/body.stl" scale="0.001 0.001 0.001"/>
             </geometry>
             <material name="">
@@ -62,7 +62,7 @@
                 <mass value="0.00001"/>
                 <inertia
-                    ixx="1.0" ixy="0.0"  ixz="0.0"
-                    iyy="1.0" iyz="0.0"
-                    izz="1.0" />
+                    ixx="0.2" ixy="0.0"  ixz="0.0"
+                    iyy="0.2" iyz="0.0"
+                    izz="0.2" />
             </inertial>
         </link>
@@ -87,7 +87,7 @@
         <link name="coxa_${side}${position}">
             <visual>
-                <origin xyz="0.0 0.0 0.0" rpy="0.0 ${pi/2} 0.0"/>
-                <geometry>
-                    <cylinder radius="0.020" length="${coxa_length}"/>
+                <origin xyz="0.0 0.0 0.0" rpy="0.0 0.0 0.0"/>
+                <geometry>
+                    <mesh filename="package://hexpet/meshes/phantomX/coxa.stl" scale="0.001 0.001 0.001"/>
                 </geometry>
                 <material name="">
@@ -108,7 +108,7 @@
                 <mass value="0.00001"/>
                 <inertia
-                    ixx="1.0" ixy="0.0"  ixz="0.0"
-                    iyy="1.0" iyz="0.0"
-                    izz="1.0" />
+                    ixx="0.01" ixy="0.0"  ixz="0.0"
+                    iyy="0.01" iyz="0.0"
+                    izz="0.01" />
             </inertial>
         </link>
@@ -136,7 +136,7 @@
         <link name="femur_${side}${position}">
             <visual>
-                <origin xyz="0.0 0.0 0.0" rpy="${pi/2} 0.0 0.0"/>
-                <geometry>
-                    <cylinder radius="0.025" length="${femur_length}"/>
+                <origin xyz="0.0 0.0 0.0" rpy="0.0 0.0 0.0"/>
+                <geometry>
+                    <mesh filename="package://hexpet/meshes/phantomX/femur.stl" scale="0.001 0.001 0.001"/>
                 </geometry>
                 <material name="">
@@ -157,7 +157,7 @@
                 <mass value="0.00001"/>
                 <inertia
-                    ixx="1.0" ixy="0.0"  ixz="0.0"
-                    iyy="1.0" iyz="0.0"
-                    izz="1.0" />
+                    ixx="0.01" ixy="0.0"  ixz="0.0"
+                    iyy="0.01" iyz="0.0"
+                    izz="0.01" />
             </inertial>
         </link>
@@ -185,7 +185,7 @@
         <link name="tibia_${side}${position}">
             <visual>
-                <origin xyz="${tibia_length/2} 0.0 0.0" rpy="${pi/2} 0.0 ${pi/2}"/>
-                <geometry>
-                    <cylinder radius="0.025" length="${tibia_length}"/>
+                <origin xyz="0.0 0.0 0.0" rpy="0.0 0.0 0.0"/>
+                <geometry>
+                    <mesh filename="package://hexpet/meshes/phantomX/tibia.stl" scale="0.001 0.001 0.001"/>
                 </geometry>
                 <material name="">
@@ -206,7 +206,7 @@
                 <mass value="0.00001"/>
                 <inertia
-                    ixx="1.0" ixy="0.0"  ixz="0.0"
-                    iyy="1.0" iyz="0.0"
-                    izz="1.0" />
+                    ixx="0.01" ixy="0.0"  ixz="0.0"
+                    iyy="0.01" iyz="0.0"
+                    izz="0.01" />
             </inertial>
         </link>

Commit message: fixed performance issues tuned inertia and related parameters

File: urdf/hexpet.xacro (robot description, xacro)
@@ -26,5 +26,5 @@
             <origin xyz="0.0 0.0 0.0" rpy="0.0 0.0 0.0"/>
             <geometry>
-                <box size="${body_length_x} ${body_length_y} 0.1"/>
+                <box size="${body_length_x} ${body_length_y} 0.025"/>
             </geometry>
             <material name="">
@@ -60,5 +60,5 @@
             <inertial>
                 <origin xyz="0.0 0.0 0.0" rpy="0.0 0.0 0.0" />
-                <mass value="0.00001"/>
+                <mass value="1.0"/>
                 <inertia
                     ixx="0.2" ixy="0.0"  ixz="0.0"
@@ -106,5 +106,5 @@
             <inertial>
                 <origin xyz="0.0 0.0 0.0" rpy="0.0 0.0 0.0" />
-                <mass value="0.00001"/>
+                <mass value="0.1"/>
                 <inertia
                     ixx="0.01" ixy="0.0"  ixz="0.0"
@@ -155,5 +155,5 @@
             <inertial>
                 <origin xyz="0.0 0.0 0.0" rpy="0.0 0.0 0.0" />
-                <mass value="0.00001"/>
+                <mass value="0.1"/>
                 <inertia
                     ixx="0.01" ixy="0.0"  ixz="0.0"
@@ -194,7 +194,7 @@
             </visual>
             <collision>
-                <origin xyz="${tibia_length/2} 0.0 0.0" rpy="${pi/2} 0.0 ${pi/2}" />
-                <geometry>
-                    <cylinder radius="0.025" length="${tibia_length}"/>
+                <origin xyz="${tibia_length/2} 0.025 0.0" rpy="${pi/2} 0.0 ${pi/2}" />
+                <geometry>
+                    <cylinder radius="0.001" length="${tibia_length}"/>
                 </geometry>
                 <material name="">
@@ -204,5 +204,5 @@
             <inertial>
                 <origin xyz="0.0 0.0 0.0" rpy="0.0 0.0 0.0" />
-                <mass value="0.00001"/>
+                <mass value="0.1"/>
                 <inertia
                     ixx="0.01" ixy="0.0"  ixz="0.0"

Commit message: fixed inertia, mass, speed, torque/force values

File: urdf/hexpet.xacro (robot description, xacro)
@@ -47,6 +47,6 @@
 	<xacro:property name="joint_lower_limit" value="-${1.57}" />
 	<xacro:property name="joint_upper_limit" value="${1.57}" />
-	<xacro:property name="joint_effort" value="6.0" />
-	<xacro:property name="joint_velocity" value="0.524" />
+	<xacro:property name="joint_effort" value="1.667" />
+	<xacro:property name="joint_velocity" value="5.24" />
 	<!-- Leg macro -->
 	<xacro:macro name="leg" params="side position x y angle axis">
@@ -60,9 +60,9 @@
             <inertial>
                 <origin xyz="0.0 0.0 0.0" rpy="0.0 0.0 0.0" />
-                <mass value="1.0"/>
-                <inertia
-                    ixx="0.2" ixy="0.0"  ixz="0.0"
-                    iyy="0.2" iyz="0.0"
-                    izz="0.2" />
+                <mass value="0.1"/>
+                <inertia
+                    ixx="0.0002" ixy="0.0"  ixz="0.0"
+                    iyy="0.0002" iyz="0.0"
+                    izz="0.0002" />
             </inertial>
         </link>
@@ -108,7 +108,7 @@
                 <mass value="0.1"/>
                 <inertia
-                    ixx="0.01" ixy="0.0"  ixz="0.0"
-                    iyy="0.01" iyz="0.0"
-                    izz="0.01" />
+                    ixx="0.0001" ixy="0.0"  ixz="0.0"
+                    iyy="0.0001" iyz="0.0"
+                    izz="0.0001" />
             </inertial>
         </link>
@@ -157,7 +157,7 @@
                 <mass value="0.1"/>
                 <inertia
-                    ixx="0.01" ixy="0.0"  ixz="0.0"
-                    iyy="0.01" iyz="0.0"
-                    izz="0.01" />
+                    ixx="0.0001" ixy="0.0"  ixz="0.0"
+                    iyy="0.0001" iyz="0.0"
+                    izz="0.0001" />
             </inertial>
         </link>
@@ -206,7 +206,7 @@
                 <mass value="0.1"/>
                 <inertia
-                    ixx="0.01" ixy="0.0"  ixz="0.0"
-                    iyy="0.01" iyz="0.0"
-                    izz="0.01" />
+                    ixx="0.0001" ixy="0.0"  ixz="0.0"
+                    iyy="0.0001" iyz="0.0"
+                    izz="0.0001" />
             </inertial>
         </link>

Commit message: commands without start up routine

File: urdf/hexpet.xacro (robot description, xacro)
@@ -47,6 +47,5 @@
 	<xacro:property name="joint_lower_limit" value="-${1.57}" />
 	<xacro:property name="joint_upper_limit" value="${1.57}" />
-	<!-- <xacro:property name="joint_effort" value="1.667" /> -->
-    <xacro:property name="joint_effort" value="100" />
+	<xacro:property name="joint_effort" value="9" />
 	<xacro:property name="joint_velocity" value="5.24" />
 	<!-- Leg macro -->
@@ -100,4 +99,5 @@
                 <geometry>
                     <cylinder radius="0.025" length="${coxa_length}"/>
+                    <cylinder radius="0.015" length="${coxa_length}"/>
                 </geometry>
                 <material name="">
